File: memory-phone-pcb/memory-phone-pcb.kicad_sch (KiCad schematic)
At the start: 0 parts

Commit message: sch work adding rp2040
Parts:
- added C? (x2): 10pF, Capacitor_SMD:C_0603_1608Metric_Pad1.08x0.95mm_HandSolder, symbol Device:C_Small
- added R?: 1k, Resistor_SMD:R_0603_1608Metric_Pad0.98x0.95mm_HandSolder, symbol Device:R
- added U?: RP2040, MCU_RaspberryPi_and_Boards:RP2040-QFN-56, symbol MCU_RaspberryPi_and_Boards:RP2040
- added U?: W25Q16JVSSIQ, MemoryPhone_footprints:W25Q16JVSSIQ, symbol MemoryPhone_sym:W25Q16JVSSIQ
- added Y?: ECS-120-8-36B-CWY-TR, MemoryPhone_footprints:XTAL_ECS-120-8-36B-CWY-TR, symbol MemoryPhone_sym:ECS-120-8-36B-CWY-TR
Connections:
- new net: C?.1, R?.1, Y?.3 (OUT/IN)
- new net: R?.2, U?.21 (XOUT)
- new net: C?.2, U?.20 (XIN), Y?.1 (IN/OUT)
- new net GND: C?.1, C?.2, Y?.2 (GND), Y?.4 (GND)
- new net QSPI_SCLK: U?.52 (QSPI_SCLK), U?.6 (CLK)
- new net QSPI_SD0: U?.5 (DI(ID0)), U?.53 (QSPI_SD0)
- new net QSPI_SD1: U?.2 (D0(IO1)), U?.55 (QSPI_SD1)
- new net QSPI_SD2: U?.3 (~{WP}(IO2)), U?.54 (QSPI_SD2)
- new net QSPI_SD3: U?.51 (QSPI_SD3), U?.7 (~{HOLD/RST}(IO3))
- new net QSPI_SS: U?.1 (~{CS}), U?.56 (QSPI_SS)
