File: memory-phone-pcb/memory-phone-pcb.kicad_sch (KiCad schematic)
At the start: 6 parts

Commit message: finished pcb
Parts:
- removed C? (x2): 10pF, Capacitor_SMD:C_0603_1608Metric_Pad1.08x0.95mm_HandSolder, symbol Device:C_Small
- removed R?: 1k, Resistor_SMD:R_0603_1608Metric_Pad0.98x0.95mm_HandSolder, symbol Device:R
- removed U?: RP2040, MCU_RaspberryPi_and_Boards:RP2040-QFN-56, symbol MCU_RaspberryPi_and_Boards:RP2040
- removed U?: W25Q16JVSSIQ, MemoryPhone_footprints:W25Q16JVSSIQ, symbol MemoryPhone_sym:W25Q16JVSSIQ
- removed Y?: ECS-120-8-36B-CWY-TR, MemoryPhone_footprints:XTAL_ECS-120-8-36B-CWY-TR, symbol MemoryPhone_sym:ECS-120-8-36B-CWY-TR
- added C1, C2, C7: 10nF, Capacitor_SMD:C_0603_1608Metric_Pad1.08x0.95mm_HandSolder, symbol Device:C_Small
- added C3: 0.1uF, Capacitor_SMD:C_0603_1608Metric_Pad1.08x0.95mm_HandSolder, symbol Device:C_Small
- added C4, C5, C6: 100nF, Capacitor_SMD:C_0603_1608Metric_Pad1.08x0.95mm_HandSolder, symbol Device:C_Small
- added C8: 2.2uF, Capacitor_SMD:C_0603_1608Metric_Pad1.08x0.95mm_HandSolder, symbol Device:C_Small
- added J1, J2: Conn_01x04, Connector_PinSocket_2.54mm:PinSocket_1x04_P2.54mm_Vertical, symbol Connector_Generic:Conn_01x04
- added J3: DM3D-SF, MemoryPhone_footprints:DM3D-SF, symbol MemoryPhone_sym:DM3D-SF
- added R1: 22R, Resistor_SMD:R_0603_1608Metric_Pad0.98x0.95mm_HandSolder, symbol Device:R
- added R2, R3, R4, R6, R8, R9: 10kR, Resistor_SMD:R_0603_1608Metric_Pad0.98x0.95mm_HandSolder, symbol Device:R
- added R5: 200R, Resistor_SMD:R_0603_1608Metric_Pad0.98x0.95mm_HandSolder, symbol Device:R
- added R7: 1MR, Resistor_SMD:R_0603_1608Metric_Pad0.98x0.95mm_HandSolder, symbol Device:R
- added RV1: TC33X-1-102E, MemoryPhone_footprints:TC33X-1, symbol Device:R_Potentiometer
- added U1: OPA196xDBV, Package_TO_SOT_SMD:SOT-23-5, symbol Amplifier_Operational:OPA196xDBV
- added U2: SN74AHCT1G125DBVR, Package_TO_SOT_SMD:SOT-23-5_HandSoldering, symbol MemoryPhone_sym:SN74AHCT1G125DBVR
- added U3: LP2985-1.5, Package_TO_SOT_SMD:SOT-23-5, symbol Regulator_Linear:LP2985-1.8
- added U4: Pico, MCU_RaspberryPi_and_Boards:RPi_Pico_SMD_TH, symbol MCU_RaspberryPi_and_Boards:Pico
- added U5: LM4040DBZ-3, Package_TO_SOT_SMD:SOT-23, symbol Reference_Voltage:LM4040DBZ-3
Connections:
- net GND: now also C3.1, C4.1, C5.1, C6.1, C7.1, C8.1, J1.2 (Pin_2), J1.4 (Pin_4), J2.2 (Pin_2), J2.4 (Pin_4), J3.10 (GND), J3.11 (GND), J3.12 (GND), J3.13 (GND), J3.14 (GND), J3.6, J3.9 (GND), U1.2 (V-), U2.1 (~{OE}), U2.3 (GND), U3.2 (GND), U4.13 (GND), U4.18 (GND), U4.23 (GND), U4.28 (GND), U4.3 (GND), U4.38 (GND), U4.8 (GND), U5.2 (A)
- new net: C2.1, J1.3 (Pin_3)
- new net: C1.1, J1.1 (Pin_1), RV1.3
- new net: J3.5, R1.1
- new net: R5.2, U2.4 (Y)
- new net: C7.2, U3.4 (BP)
- new net +1V5: C8.2, R7.1, U3.5 (VOUT)
- new net +3V3: C3.2, C4.2, C5.2, C6.2, J3.4, R2.1, R3.1, R4.1, R6.1, R8.1, R9.1, RV1.1, RV1.2, U1.5 (V+), U2.5 (VCC), U3.1 (VIN), U3.3 (ON/~{OFF}), U4.36 (3V3)
- new net +5V: U4.40 (VBUS)
- new net ADC_VREF: U4.35 (ADC_VREF), U5.1 (K)
- new net DIAL: J2.3 (Pin_3), R9.2, U4.19 (GPIO14)
- new net HANDSET_ADC_IN: U1.1, U1.4 (-), U4.31 (GPIO26_ADC0)
- new net HANDSET_MIC_IN: C1.2, R7.2, U1.3 (+)
- new net HANDSET_PWM_OUT: U2.2 (A), U4.29 (GPIO22)
- new net HANDSET_SPEAKER_OUT: C2.2, R5.1
- new net HANG_UP: J2.1 (Pin_1), R8.2, U4.20 (GPIO15)
- new net SD_CSn: J3.2, R2.2, U4.22 (GPIO17)
- new net SD_SCK: R1.2, R4.2, U4.24 (GPIO18)
- new net SD_SDI: J3.3, R3.2, U4.25 (GPIO19)
- new net SD_SDO: J3.7, R6.2, U4.21 (GPIO16)
- no-connect marks 0 -> 25
